Commit message: added initail to joints in urdf

File: envs/stoch3/urdf/stoch3.urdf (robot description, URDF)
Before this commit: robot stoch3, 13 links, 12 joints
Links:
- link motor_back_right_abd_link: mass 1.702 -> 4.11
- link motor_fl_upper_hip_link: mass 1.56 -> 1.561
- link motor_front_left_abd_link: mass 1702 -> 1.702
Joints:
- joint motor_back_left_abd_joint: limit lower=0 upper=0 effort=0 velocity=0 -> lower=-0.34907 upper=3.4907 effort=30 velocity=100
- joint motor_back_right_abd_joint: limit lower=0 upper=0 effort=0 velocity=0 -> lower=0.34907 upper=-3.4907 effort=30 velocity=100
- joint motor_bl_upper_hip_joint: limit lower=0 upper=0 effort=0 velocity=0 -> lower=-12.566 upper=12.566 effort=30 velocity=100
- joint motor_bl_upper_knee_joint: limit lower=0 upper=0 effort=0 velocity=0 -> lower=-12.566 upper=12.566 effort=30 velocity=100
- joint motor_br_upper_hip_joint: limit lower=0 upper=0 effort=0 velocity=0 -> lower=-12.566 upper=12.566 effort=30 velocity=100; origin xyz=-0.0844999999999999 -0.0624999999999987 0 rpy=0 0 0 -> xyz=-0.0845 -0.0625 0 rpy=0 0 0
- joint motor_br_upper_knee_joint: limit lower=0 upper=0 effort=0 velocity=0 -> lower=-12.566 upper=12.566 effort=30 velocity=100; origin xyz=-0.192307885658796 -0.0554999999998631 -0.230255677700808 rpy=0 0 0 -> xyz=-0.19231 -0.0555 -0.23026 rpy=0 0 0
- joint motor_fl_upper_hip_joint: limit lower=0 upper=0 effort=0 velocity=0 -> lower=-12.566 upper=12.566 effort=30 velocity=100
- joint motor_fl_upper_knee_joint: limit lower=0 upper=0 effort=0 velocity=0 -> lower=-12.566 upper=12.566 effort=30 velocity=100
- joint motor_fr_upper_hip_joint: limit lower=0 upper=0 effort=0 velocity=0 -> lower=-12.566 upper=12.566 effort=30 velocity=100
- joint motor_fr_upper_knee_joint: limit lower=0 upper=0 effort=0 velocity=0 -> lower=-12.566 upper=12.566 effort=30 velocity=100
- joint motor_front_left_abd_joint: limit lower=0 upper=0 effort=0 velocity=0 -> lower=-0.34907 upper=3.4907 effort=30 velocity=100
- joint motor_front_right_abd_joint: limit lower=0 upper=0 effort=0 velocity=0 -> lower=0.34907 upper=-3.4907 effort=30 velocity=100

Commit message: removed urdf file

File: envs/stoch3/urdf/stoch3.urdf (robot description, URDF)
Before this commit: robot stoch3, 13 links, 12 joints
Links:
- link motor_back_right_abd_link: mass 4.11 -> 1.702
- link motor_fl_upper_hip_link: mass 1.561 -> 1.56
- link motor_front_left_abd_link: mass 1.702 -> 1702
Joints:
- joint motor_back_left_abd_joint: limit lower=-0.34907 upper=3.4907 effort=30 velocity=100 -> lower=0 upper=0 effort=0 velocity=0
- joint motor_back_right_abd_joint: limit lower=0.34907 upper=-3.4907 effort=30 velocity=100 -> lower=0 upper=0 effort=0 velocity=0
- joint motor_bl_upper_hip_joint: limit lower=-12.566 upper=12.566 effort=30 velocity=100 -> lower=0 upper=0 effort=0 velocity=0
- joint motor_bl_upper_knee_joint: limit lower=-12.566 upper=12.566 effort=30 velocity=100 -> lower=0 upper=0 effort=0 velocity=0
- joint motor_br_upper_hip_joint: limit lower=-12.566 upper=12.566 effort=30 velocity=100 -> lower=0 upper=0 effort=0 velocity=0; origin xyz=-0.0845 -0.0625 0 rpy=0 0 0 -> xyz=-0.0844999999999999 -0.0624999999999987 0 rpy=0 0 0
- joint motor_br_upper_knee_joint: limit lower=-12.566 upper=12.566 effort=30 velocity=100 -> lower=0 upper=0 effort=0 velocity=0; origin xyz=-0.19231 -0.0555 -0.23026 rpy=0 0 0 -> xyz=-0.192307885658796 -0.0554999999998631 -0.230255677700808 rpy=0 0 0
- joint motor_fl_upper_hip_joint: limit lower=-12.566 upper=12.566 effort=30 velocity=100 -> lower=0 upper=0 effort=0 velocity=0
- joint motor_fl_upper_knee_joint: limit lower=-12.566 upper=12.566 effort=30 velocity=100 -> lower=0 upper=0 effort=0 velocity=0
- joint motor_fr_upper_hip_joint: limit lower=-12.566 upper=12.566 effort=30 velocity=100 -> lower=0 upper=0 effort=0 velocity=0
- joint motor_fr_upper_knee_joint: limit lower=-12.566 upper=12.566 effort=30 velocity=100 -> lower=0 upper=0 effort=0 velocity=0
- joint motor_front_left_abd_joint: limit lower=-0.34907 upper=3.4907 effort=30 velocity=100 -> lower=0 upper=0 effort=0 velocity=0
- joint motor_front_right_abd_joint: limit lower=0.34907 upper=-3.4907 effort=30 velocity=100 -> lower=0 upper=0 effort=0 velocity=0
